File: Europe-ergo-PCB/Europe-ergo.kicad_sch (KiCad schematic)
At the start: 230 parts, among them J1 SJ-43514, J2 SJ-43514, SW1 MX1A-G1NN, SW10 MX1A-G1NN, SW11 MX1A-G1NN, SW12 MX1A-G1NN, SW13 MX1A-G1NN, SW14 MX1A-G1NN, SW15 MX1A-G1NN, SW16 MX1A-G1NN, SW17 MX1A-G1NN, SW18 MX1A-G1NN, SW19 MX1A-G1NN, SW2 MX1A-G1NN, SW20 MX1A-G1NN, SW21 MX1A-G1NN, SW22 MX1A-G1NN, SW23 MX1A-G1NN, SW24 MX1A-G1NN, SW25 MX1A-G1NN, SW26 MX1A-G1NN, SW27 MX1A-G1NN, SW28 MX1A-G1NN, SW29 MX1A-G1NN, SW3 MX1A-G1NN, SW30 MX1A-G1NN, SW31 MX1A-G1NN, SW32 MX1A-G1NN, SW33 MX1A-G1NN, SW34 MX1A-G1NN, SW35 MX1A-G1NN, SW36 MX1A-G1NN, SW37 MX1A-G1NN, SW38 MX1A-G1NN, SW39 MX1A-G1NN, SW4 MX1A-G1NN, SW40 MX1A-G1NN, SW41 MX1A-G1NN, SW42 MX1A-G1NN, SW43 MX1A-G1NN, SW44 MX1A-G1NN, SW45 MX1A-G1NN, SW46 MX1A-G1NN, SW47 MX1A-G1NN, SW48 800SP9B6M2RE, SW49 800SP9B6M2RE, SW5 MX1A-G1NN, SW50 MX1A-G1NN, SW51 MX1A-G1NN, SW52 MX1A-G1NN, SW53 MX1A-G1NN, SW54 MX1A-G1NN, SW55 MX1A-G1NN, SW56 MX1A-G1NN, SW57 MX1A-G1NN, SW58 MX1A-G1NN, SW59 MX1A-G1NN, SW6 MX1A-G1NN, SW60 MX1A-G1NN, SW61 MX1A-G1NN, SW62 MX1A-G1NN, SW63 MX1A-G1NN, SW64 MX1A-G1NN, SW65 MX1A-G1NN, SW66 MX1A-G1NN, SW67 MX1A-G1NN, SW68 MX1A-G1NN, SW69 MX1A-G1NN, SW7 MX1A-G1NN, SW70 MX1A-G1NN, SW71 MX1A-G1NN, SW72 MX1A-G1NN, SW73 MX1A-G1NN, SW74 MX1A-G1NN, SW75 MX1A-G1NN, SW76 MX1A-G1NN, SW77 MX1A-G1NN, SW78 MX1A-G1NN, SW79 MX1A-G1NN, SW8 MX1A-G1NN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

Commit message: Add files via upload
Parts:
- renumbered D102 to D1, D13 to D10, D83 to D100, D30 to D101, D24 to D102, D84 to D11, D78 to D12, D25 to D13, D19 to D14, D100 to D15, D92 to D16, D60 to D17, D42 to D18, D8 to D19, D96 to D2, D2 to D20, D87 to D21, D79 to D22, D73 to D23, D68 to D24, D64 to D25, D38 to D26, D32 to D27, D27 to D28, D20 to D29, D90 to D3, D14 to D30, D55 to D31, D54 to D32, D101 to D33, D93 to D34, D59 to D35, D53 to D36, D52 to D37, D48 to D38, D49 to D39, D72 to D4, D50 to D40, D51 to D41, D43 to D42, D9 to D43, D3 to D44, D69 to D45, D62 to D46, D88 to D47, D40 to D48, D33 to D49, D66 to D5, D80 to D50, D77 to D51, D15 to D52, D26 to D53, D21 to D54, D98 to D55, D94 to D56, D10 to D57, D4 to D58, D74 to D59, D7 to D6, D70 to D60, D63 to D61, D85 to D62, D81 to D63, D41 to D64, D34 to D65, D28 to D66, D22 to D67, D17 to D68, D99 to D69, D1 to D7, D95 to D70, D58 to D71, D57 to D72, D46 to D73, D45 to D74, D11 to D75, D5 to D76, D89 to D77, D82 to D78, D75 to D79, D37 to D8, D71 to D80, D35 to D81, D29 to D82, D23 to D83, D16 to D84, D65 to D85, D39 to D86, D97 to D87, D91 to D88, D67 to D89, D31 to D9, D61 to D90, D56 to D91, D47 to D92, D44 to D93, D36 to D94, D12 to D95, D6 to D96, D86 to D97, D76 to D98, D18 to D99, H9 to H1, H5 to H10, H14 to H11, H6 to H12, H15 to H13, H7 to H14, H16 to H15, H8 to H16, H1 to H2, H10 to H3, H2 to H4, H11 to H5, H3 to H6, H12 to H7, H4 to H8, H13 to H9, J2 to J1, J1 to J2, R12 to R1, R5 to R10, R9 to R11, R11 to R12, R10 to R2, R8 to R3, R7 to R4, R1 to R5, R2 to R6, R4 to R7, R6 to R8, R3 to R9, SW96 to SW1, SW25 to SW10, SW19 to SW11, SW13 to SW12, SW7 to SW13, SW1 to SW14, SW49 to SW15, SW48 to SW16, SW93 to SW17, SW87 to SW18, SW81 to SW19, SW90 to SW2, SW75 to SW20, SW69 to SW21, SW62 to SW22, SW57 to SW23, SW52 to SW24, SW42 to SW25, SW38 to SW26, SW32 to SW27, SW26 to SW28, SW20 to SW29, SW84 to SW3, SW14 to SW30, SW8 to SW31, SW2 to SW32, SW94 to SW33, SW88 to SW34, SW82 to SW35, SW76 to SW36, SW70 to SW37, SW63 to SW38, SW58 to SW39, SW78 to SW4, SW53 to SW40, SW43 to SW41, SW39 to SW42, SW33 to SW43, SW27 to SW44, SW21 to SW45, SW15 to SW46, SW9 to SW47, SW3 to SW48, SW91 to SW49, SW72 to SW5, SW85 to SW50, SW79 to SW51, SW73 to SW52, SW67 to SW53, SW61 to SW54, SW56 to SW55, SW41 to SW56, SW36 to SW57, SW29 to SW58, SW23 to SW59, SW66 to SW6, SW17 to SW60, SW11 to SW61, SW5 to SW62, SW95 to SW63, SW89 to SW64, SW83 to SW65, SW77 to SW66, SW71 to SW67, SW64 to SW68, SW59 to SW69, SW60 to SW7, SW54 to SW70, SW51 to SW71, SW46 to SW72, SW44 to SW73, SW40 to SW74, SW34 to SW75, SW28 to SW76, SW22 to SW77, SW16 to SW78, SW10 to SW79, SW37 to SW8, SW4 to SW80, SW92 to SW81, SW86 to SW82, SW80 to SW83, SW74 to SW84, SW68 to SW85, SW65 to SW86, SW55 to SW87, SW50 to SW88, SW47 to SW89, SW31 to SW9, SW45 to SW90, SW35 to SW91, SW30 to SW92, SW24 to SW93, SW18 to SW94, SW12 to SW95, SW6 to SW96, U2 to U1, U1 to U2

Commit message: Add files via upload
Parts:
- added D38, D43: LTL-4233, Diode_THT:D_A-405_P2.54mm_Vertical_AnodeUp, symbol Device:LED
- added R10, R5: 330, Resistor_THT:R_Axial_DIN0204_L3.6mm_D1.6mm_P5.08mm_Horizontal, symbol Device:R
- renumbered D98 to D100, D99 to D101, D100 to D102, D101 to D103, D102 to D104, D38 to D39, D39 to D40, D40 to D41, D41 to D42, D42 to D44, D43 to D45, D44 to D46, D45 to D47, D46 to D48, D47 to D49, D48 to D50, D49 to D51, D50 to D52, D51 to D53, D52 to D54, D53 to D55, D54 to D56, D55 to D57, D56 to D58, D57 to D59, D58 to D60, D59 to D61, D60 to D62, D61 to D63, D62 to D64, D63 to D65, D64 to D66, D65 to D67, D66 to D68, D67 to D69, D68 to D70, D69 to D71, D70 to D72, D71 to D73, D72 to D74, D73 to D75, D74 to D76, D75 to D77, D76 to D78, D77 to D79, D78 to D80, D79 to D81, D80 to D82, D81 to D83, D82 to D84, D83 to D85, D84 to D86, D85 to D87, D86 to D88, D87 to D89, D88 to D90, D89 to D91, D90 to D92, D91 to D93, D92 to D94, D93 to D95, D94 to D96, D95 to D97, D96 to D98, D97 to D99, R9 to R11, R10 to R12, R11 to R13, R12 to R14, R5 to R6, R6 to R7, R7 to R8, R8 to R9
Connections:
- net GNDL: now also R5.1
- net GNDR: now also R10.1
- net PWM5R: now reaches U2.29 (GPIO22)
- net PWM5R: now also D43.2 (A)
- net PWM5: now reaches U1.29 (GPIO22)
- net PWM5: now also D38.2 (A)
- new net: D43.1 (K), R10.2
- new net: D38.1 (K), R5.2
- no-connect marks 21 -> 19
Other:
- note added: "NUM"
- note added: "OMIT 4.7K RES IF SERIAL COMM IS USED."
- note removed: "OMIT R9 R11 IF SERIAL COMM IS USED."
