File: Europe-ergo-smd/europe-ergo-smd/europe-ergo-smd.kicad_sch (KiCad schematic)
At the start: 230 parts, among them J1 SJ-43514, J2 SJ-43514, SW1 MX1A-G1NN, SW10 MX1A-G1NN, SW11 MX1A-G1NN, SW12 MX1A-G1NN, SW13 MX1A-G1NN, SW14 MX1A-G1NN, SW15 MX1A-G1NN, SW16 MX1A-G1NN, SW17 MX1A-G1NN, SW18 MX1A-G1NN, SW19 MX1A-G1NN, SW2 MX1A-G1NN, SW20 MX1A-G1NN, SW21 MX1A-G1NN, SW22 MX1A-G1NN, SW23 MX1A-G1NN, SW24 MX1A-G1NN, SW25 MX1A-G1NN, SW26 MX1A-G1NN, SW27 MX1A-G1NN, SW28 MX1A-G1NN, SW29 MX1A-G1NN, SW3 MX1A-G1NN, SW30 MX1A-G1NN, SW31 MX1A-G1NN, SW32 MX1A-G1NN, SW33 MX1A-G1NN, SW34 MX1A-G1NN, SW35 MX1A-G1NN, SW36 MX1A-G1NN, SW37 MX1A-G1NN, SW38 MX1A-G1NN, SW39 MX1A-G1NN, SW4 MX1A-G1NN, SW40 MX1A-G1NN, SW41 MX1A-G1NN, SW42 MX1A-G1NN, SW43 MX1A-G1NN, SW44 MX1A-G1NN, SW45 MX1A-G1NN, SW46 MX1A-G1NN, SW47 MX1A-G1NN, SW48 800SP9B6M2RE, SW49 800SP9B6M2RE, SW5 MX1A-G1NN, SW50 MX1A-G1NN, SW51 MX1A-G1NN, SW52 MX1A-G1NN, SW53 MX1A-G1NN, SW54 MX1A-G1NN, SW55 MX1A-G1NN, SW56 MX1A-G1NN, SW57 MX1A-G1NN, SW58 MX1A-G1NN, SW59 MX1A-G1NN, SW6 MX1A-G1NN, SW60 MX1A-G1NN, SW61 MX1A-G1NN, SW62 MX1A-G1NN, SW63 MX1A-G1NN, SW64 MX1A-G1NN, SW65 MX1A-G1NN, SW66 MX1A-G1NN, SW67 MX1A-G1NN, SW68 MX1A-G1NN, SW69 MX1A-G1NN, SW7 MX1A-G1NN, SW70 MX1A-G1NN, SW71 MX1A-G1NN, SW72 MX1A-G1NN, SW73 MX1A-G1NN, SW74 MX1A-G1NN, SW75 MX1A-G1NN, SW76 MX1A-G1NN, SW77 MX1A-G1NN, SW78 MX1A-G1NN, SW79 MX1A-G1NN, SW8 MX1A-G1NN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

Commit message: Add files via upload
Parts:
- D1, D10, D100, D101, D102, D11, D12, D13, D14, D15, D16, D17, D18, D19, D2, D20, D21, D22, D23, D24, D25, D26, D27, D28, D29, D3, D30, D31, D32, D33, D34, D35, D36, D37, D38, D39, D4, D40, D41, D42, D43, D44, D45, D46, D47, D5, D56, D57, D58, D59, D6, D60, D61, D62, D63, D64, D65, D66, D67, D68, D69, D7, D70, D71, D72, D73, D74, D75, D76, D77, D78, D79, D8, D80, D81, D82, D83, D84, D85, D86, D87, D88, D89, D9, D90, D91, D92, D93, D94, D95, D96, D97, D98, D99: value 1N4148W-13-F -> 1N4148W
- R1, R10, R11, R12, R2, R3, R4, R5, R6, R7, R8, R9: footprint Resistor_SMD:R_2512_6332Metric -> Resistor_SMD:R_1812_4532Metric
